Commit message: Add table in the map.

File: iai_kitchen/urdf/IAI_kitchen.urdf.xacro (robot description, xacro)
@@ -28,11 +28,12 @@
   </gazebo>
   <!--- FIXME THIS should NOT be here -->
-  <xacro:include filename="$(find iai_kitchen)/urdf/IAI_oven_area.urdf.xacro"/>
+  <!-- <xacro:include filename="$(find iai_kitchen)/urdf/IAI_oven_area.urdf.xacro"/>
   <xacro:include filename="$(find iai_kitchen)/urdf/IAI_kitchen_island.urdf.xacro"/>
   <xacro:include filename="$(find iai_kitchen)/urdf/IAI_sink_area.urdf.xacro"/>
   <xacro:include filename="$(find iai_kitchen)/urdf/IAI_fridge_area.urdf.xacro"/>
-  <xacro:include filename="$(find iai_kitchen)/urdf/IAI_tables.urdf.xacro"/>
-  <xacro:include filename="$(find iai_kitchen)/urdf/IAI_kitchen_walls.urdf.xacro"/>
-  <iai_sink_area name="sink_area" parent="room_link">
+   -->
+   <xacro:include filename="$(find iai_kitchen)/urdf/IAI_tables.urdf.xacro"/>
+  <!-- <xacro:include filename="$(find iai_kitchen)/urdf/IAI_kitchen_walls.urdf.xacro"/> -->
+  <!-- <iai_sink_area name="sink_area" parent="room_link">
     <origin xyz="1.825 1.32 0" rpy="0 0 ${pi}" />
   </iai_sink_area>
@@ -45,11 +46,13 @@
   <iai_fridge_area name="fridge_area" parent="room_link">
     <origin xyz="1.825 -0.74 0" rpy="0 0 ${pi}" />
-  </iai_fridge_area>
+  </iai_fridge_area> -->
   <iai_table_1 name="table_area" parent="room_link">
-    <origin xyz="-1.4 -1.05 0" rpy="0 0 ${pi}" />
+    <origin xyz="-0.35 -1.7 0" rpy="0 0 ${pi}" />
   </iai_table_1>
-  <iai_kitchen_wall_robohow parent="room_link">
+  <!-- 80cm, 80cm, 71,7cm -->
+  <!-- 6, 24,7 80 116,2 147,8-->
+  <!-- <iai_kitchen_wall_robohow parent="room_link">
     <origin xyz="-1 0.562175 0" rpy="0.0 0.0 0.0" />
-  </iai_kitchen_wall_robohow>
+  </iai_kitchen_wall_robohow> -->
   <!-- Included above already
   <iai_sink_area name="sink_area" parent="room_link">

File: iai_kitchen/urdf/IAI_tables.urdf.xacro (robot description, xacro)
@@ -8,5 +8,5 @@
         <origin xyz="0 0 0" rpy="0 0 0" />
         <geometry>
-          <mesh filename="package://iai_kitchen/meshes/misc/big_table_1.dae"/>
+          <mesh filename="package://iai_kitchen/meshes/misc/square_table.dae"/>
         </geometry>
       </visual>
@@ -14,5 +14,5 @@
         <origin xyz="0 0 0" rpy="0 0 0" />
         <geometry>
-          <mesh filename="package://iai_kitchen/meshes/misc/big_table_1.stl"/>
+          <mesh filename="package://iai_kitchen/meshes/misc/square_table.stl"/>
         </geometry>
       </collision>
