Commit message: Add xacro.urdf with data only based on semantic_map_manual_data.yaml in suturo_perception_msgs

File: iai_hsr_robocup/urdf/HSR_robocup.urdf.xacro (robot description, xacro)
@@ -1,10 +1,10 @@
 <?xml version="1.0"?>
 <robot name="kitchen_description" xmlns:xacro="http://ros.org/wiki/xacro">
-  <!-- Define data here, to make poses & dimensions easily adjustable from the outside -->
-  <xacro:property name="data" value="${load_yaml('$(find suturo_perception_msgs)/config/semantic_map_without_opencv_annotation.yaml')}" />
+  <xacro:property name="data"
+    value="${load_yaml('$(find suturo_perception_msgs)/config/semantic_map_manual_data.yaml')}" />
   <xacro:property name="table_x"
-    value="${data['robocup_table']['transform']['data'][3] - table_depth/2}" />
+    value="${data['robocup_table']['x_pos']}" />
   <xacro:property name="table_y"
-    value="${data['robocup_table']['transform']['data'][7] - table_width/2}" />
+    value="${data['robocup_table']['y_pos']}" />
   <xacro:property name="table_z_rot"
     value="${data['robocup_table']['z_rot']}" />
@@ -16,11 +16,17 @@
     value="${data['robocup_table']['height']}" />
   <xacro:property name="shelf_x"
-    value="-${shelf_width}" />
-  <xacro:property name="shelf_y" value="0.0" />
-  <xacro:property name="shelf_z_rot" value="${pi * 1.5}" />
-  <xacro:property name="shelf_depth" value="0.3" />
-  <xacro:property name="shelf_width" value="0.99" />
-  <xacro:property name="shelf_height" value="1.5" />
-  <xacro:property name="shelf_floors_height" value="[0.06, 0.247, 0.80, 1.162, 1.478]" />
+    value="${data['robocup_shelf']['x_pos']}" />
+  <xacro:property name="shelf_y"
+    value="${data['robocup_shelf']['y_pos']}" />
+  <xacro:property name="shelf_z_rot"
+    value="${data['robocup_shelf']['z_rot']}" />
+  <xacro:property name="shelf_depth"
+    value="${data['robocup_shelf']['depth']}" />
+  <xacro:property name="shelf_width"
+    value="${data['robocup_shelf']['width']}" />
+  <xacro:property name="shelf_height"
+    value="${data['robocup_shelf']['height']}" />
+  <xacro:property name="shelf_floors_height"
+    value="${data['robocup_shelf']['floors_height']}" />
   <link name="env_origin"/>
   <xacro:include filename="$(find iai_hsr_robocup)/urdf/HSR_table.urdf.xacro"/>

File: iai_hsr_robocup/urdf/HSR_shelf.urdf.xacro (robot description, xacro)
@@ -5,7 +5,63 @@
   </material>
   <macro name="robocup_shelf" params="name parent *origin size_x size_y size_z floors_height">
-    <!-- LINKS -->
-    <link name="${name}_center">
-      <!--  <sphere_inertia radius="0" mass="0"/> -->
+    <!-- General conveinience links -->
+    <link name="${name}_origin"/>
+    <link name="${name}_center"/>
+    <link name="${name}_base_center"/>
+    <joint name="${name}_origin_joint" type="fixed">
+      <xacro:insert_block name="origin" />
+      <parent link="${parent}"/>
+      <child link="${name}_origin"/>
+    </joint>
+    <joint name="${name}_center_joint" type="fixed">
+      <origin xyz="${size_x/2} ${size_y/2} ${size_z/2}" rpy="0 0 0" />
+      <parent link="${name}_origin"/>
+      <child link="${name}_center"/>
+    </joint>
+    <joint name="${name}_base_center_joint" type="fixed">
+      <origin xyz="${size_x/2} ${size_y/2} 0.0" rpy="0 0 0" />
+      <parent link="${name}_origin"/>
+      <child link="${name}_base_center"/>
+    </joint>
+    <!-- WALLS -->
+    <robocup_shelf_piece name="${name}_back" parent="${name}_origin"
+      size_x="0.08" size_y="${size_y}" size_z="${size_z}">
+      <origin xyz="${size_x} ${size_y/2} ${size_z/2}" rpy="0 0 0"/>
+    </robocup_shelf_piece>
+    <robocup_shelf_piece name="${name}_right_side" parent="${name}_origin"
+      size_x="${size_x}" size_y="0.01" size_z="${size_z}">
+      <origin xyz="${size_x/2} 0.0 ${size_z/2}" rpy="0 0 0"/>
+    </robocup_shelf_piece>
+    <robocup_shelf_piece name="${name}_left_side" parent="${name}_origin"
+      size_x="${size_x}" size_y="0.01" size_z="${size_z}">
+      <origin xyz="${size_x/2} ${size_y} ${size_z/2}" rpy="0 0 0"/>
+    </robocup_shelf_piece>
+    <!-- FLOORS -->
+    <robocup_shelf_piece name="${name}_floor_0" parent="${name}_base_center"
+      size_x="${size_x}" size_y="${size_y}" size_z="0.04">
+      <origin xyz="0.0 0.0 ${floors_height[0] - 0.02}" rpy="0 0 0"/>
+    </robocup_shelf_piece>
+    <robocup_shelf_piece name="${name}_floor_1" parent="${name}_base_center"
+      size_x="${size_x}" size_y="${size_y}" size_z="0.04">
+      <origin xyz="0.0 0.0 ${floors_height[1] - 0.02}" rpy="0 0 0"/>
+    </robocup_shelf_piece>
+    <robocup_shelf_piece name="${name}_floor_2" parent="${name}_base_center"
+      size_x="${size_x}" size_y="${size_y}" size_z="0.04">
+      <origin xyz="0.0 0.0 ${floors_height[2] - 0.02}" rpy="0 0 0"/>
+    </robocup_shelf_piece>
+    <robocup_shelf_piece name="${name}_floor_3" parent="${name}_base_center"
+      size_x="${size_x}" size_y="${size_y}" size_z="0.04">
+      <origin xyz="0.0 0.0 ${floors_height[3] - 0.02}" rpy="0 0 0"/>
+    </robocup_shelf_piece>
+    <robocup_shelf_piece name="${name}_floor_4" parent="${name}_base_center"
+      size_x="${size_x}" size_y="${size_y}" size_z="0.04">
+      <origin xyz="0.0 0.0 ${floors_height[4] - 0.02}" rpy="0 0 0"/>
+    </robocup_shelf_piece>
+  </macro>
+  <!-- Creates a link with collision and visual box of given dimensions,
+  and a respective joint to append it to the parent with given origin.  -->
+  <macro name="robocup_shelf_piece" params="name parent *origin size_x size_y size_z">
+    <!-- LINK -->
+    <link name="${name}_piece">
       <visual>
         <material name="shelf_grey"/>
@@ -22,28 +78,9 @@
       </collision>
     </link>
-    <link name="${name}_origin"/>
-    <!-- Additional tf-frames -->
-    <link name="${name}_surface_center"/>
-    <link name="${name}_front_edge_center"/>
-    <!-- JOINTS -->
-    <joint name="${name}_origin_joint" type="fixed">
+    <!-- JOINT -->
+    <joint name="${name}_piece_joint" type="fixed">
       <xacro:insert_block name="origin" />
       <parent link="${parent}"/>
-      <child link="${name}_origin"/>
-    </joint>
-    <joint name="${name}_center_joint" type="fixed">
-      <origin xyz="${size_x/2} ${size_y/2} ${size_z/2}" rpy="0 0 0" />
-      <parent link="${name}_origin"/>
-      <child link="${name}_center"/>
-    </joint>
-    <joint name="${name}_surface_center_joint" type="fixed">
-      <origin xyz="${size_x/2} ${size_y/2} ${size_z}" rpy="0 0 0" />
-      <parent link="${name}_origin"/>
-      <child link="${name}_surface_center"/>
-    </joint>
-    <joint name="${name}_front_edge_center_joint" type="fixed">
-      <origin xyz="0 ${size_y/2} ${size_z}" rpy="0 0 0" />
-      <parent link="${name}_origin"/>
-      <child link="${name}_front_edge_center"/>
+      <child link="${name}_piece"/>
     </joint>
   </macro>

Commit message: Add dynamic number of shelve floors

File: iai_hsr_robocup/urdf/HSR_robocup.urdf.xacro (robot description, xacro)
@@ -29,4 +29,6 @@
   <xacro:property name="shelf_floors_height"
     value="${data['robocup_shelf']['floors_height']}" />
+    <xacro:property name="num_floors"
+    value="${data['robocup_shelf']['num_floors']}" />
   <link name="env_origin"/>
   <xacro:include filename="$(find iai_hsr_robocup)/urdf/HSR_table.urdf.xacro"/>

File: iai_hsr_robocup/urdf/HSR_shelf.urdf.xacro (robot description, xacro)
@@ -38,24 +38,46 @@
     </robocup_shelf_piece>
     <!-- FLOORS -->
-    <robocup_shelf_piece name="${name}_floor_0" parent="${name}_base_center"
-      size_x="${size_x}" size_y="${size_y}" size_z="0.04" box_z_offset="-0.02">
-      <origin xyz="0.0 0.0 ${floors_height[0]}" rpy="0 0 0"/>
-    </robocup_shelf_piece>
-    <robocup_shelf_piece name="${name}_floor_1" parent="${name}_base_center"
-      size_x="${size_x}" size_y="${size_y}" size_z="0.04" box_z_offset="-0.02">
-      <origin xyz="0.0 0.0 ${floors_height[1]}" rpy="0 0 0"/>
-    </robocup_shelf_piece>
-    <robocup_shelf_piece name="${name}_floor_2" parent="${name}_base_center"
-      size_x="${size_x}" size_y="${size_y}" size_z="0.04" box_z_offset="-0.02">
-      <origin xyz="0.0 0.0 ${floors_height[2]}" rpy="0 0 0"/>
-    </robocup_shelf_piece>
-    <robocup_shelf_piece name="${name}_floor_3" parent="${name}_base_center"
-      size_x="${size_x}" size_y="${size_y}" size_z="0.04" box_z_offset="-0.02">
-      <origin xyz="0.0 0.0 ${floors_height[3]}" rpy="0 0 0"/>
-    </robocup_shelf_piece>
-    <robocup_shelf_piece name="${name}_floor_4" parent="${name}_base_center"
-      size_x="${size_x}" size_y="${size_y}" size_z="0.04" box_z_offset="-0.02">
-      <origin xyz="0.0 0.0 ${floors_height[4]}" rpy="0 0 0"/>
-    </robocup_shelf_piece>
+    <xacro:if value="${num_floors > 0}">
+      <robocup_shelf_piece name="${name}_floor_0" parent="${name}_base_center"
+        size_x="${size_x}" size_y="${size_y}" size_z="0.04" box_z_offset="-0.02">
+        <origin xyz="0.0 0.0 ${floors_height[0]}" rpy="0 0 0"/>
+      </robocup_shelf_piece>
+    </xacro:if>
+    <xacro:if value="${num_floors > 1}">
+      <robocup_shelf_piece name="${name}_floor_1" parent="${name}_base_center"
+        size_x="${size_x}" size_y="${size_y}" size_z="0.04" box_z_offset="-0.02">
+        <origin xyz="0.0 0.0 ${floors_height[1]}" rpy="0 0 0"/>
+      </robocup_shelf_piece>
+    </xacro:if>
+    <xacro:if value="${num_floors > 2}">
+      <robocup_shelf_piece name="${name_floor_2" parent="${name}_base_center"
+        size_x="${size_x}" size_y="${size_y}" size_z="0.04" box_z_offset="-0.02">
+        <origin xyz="0.0 0.0 ${floors_height[2]}" rpy="0 0 0"/>
+      </robocup_shelf_piece>
+    </xacro:if>
+    <xacro:if value="${num_floors > 3}">
+      <robocup_shelf_piece name="${name}_floor_3" parent="${name}_base_center"
+        size_x="${size_x}" size_y="${size_y}" size_z="0.04" box_z_offset="-0.02">
+        <origin xyz="0.0 0.0 ${floors_height[3]}" rpy="0 0 0"/>
+      </robocup_shelf_piece>
+    </xacro:if>
+    <xacro:if value="${num_floors > 4}">
+      <robocup_shelf_piece name="${name}_floor_4" parent="${name}_base_center"
+        size_x="${size_x}" size_y="${size_y}" size_z="0.04" box_z_offset="-0.02">
+        <origin xyz="0.0 0.0 ${floors_height[4]}" rpy="0 0 0"/>
+      </robocup_shelf_piece>
+    </xacro:if>
+    <xacro:if value="${num_floors > 5}">
+      <robocup_shelf_piece name="${name}_floor_5" parent="${name}_base_center"
+        size_x="${size_x}" size_y="${size_y}" size_z="0.04" box_z_offset="-0.02">
+        <origin xyz="0.0 0.0 ${floors_height[5]}" rpy="0 0 0"/>
+      </robocup_shelf_piece>
+    </xacro:if>
+    <xacro:if value="${num_floors > 6}">
+      <robocup_shelf_piece name="${name}_floor_5" parent="${name}_base_center"
+        size_x="${size_x}" size_y="${size_y}" size_z="0.04" box_z_offset="-0.02">
+        <origin xyz="0.0 0.0 ${floors_height[6]}" rpy="0 0 0"/>
+      </robocup_shelf_piece>
+    </xacro:if>
   </macro>
   <!-- Creates a link with collision and visual box of given dimensions,
