Commit message: New map with env_origin on shelf corner and table right of the shelf

File: iai_hsr_robocup/urdf/HSR_robocup.urdf (robot description, URDF)
Before this commit: robot kitchen_description, 16 links, 15 joints
Links:
- link shelf_back_piece: geometry collision box size=0.01 0.98 1.5; visual box size=0.01 0.98 1.5
- link shelf_floor_0_piece: geometry collision box size=0.36 0.98 0.04; visual box size=0.36 0.98 0.04
- link shelf_floor_1_piece: geometry collision box size=0.36 0.98 0.04; visual box size=0.36 0.98 0.04
- link shelf_floor_2_piece: geometry collision box size=0.36 0.98 0.04; visual box size=0.36 0.98 0.04
- link shelf_floor_3_piece: geometry collision box size=0.36 0.98 0.04; visual box size=0.36 0.98 0.04
- link shelf_floor_4_piece: geometry collision box size=0.36 0.98 0.04; visual box size=0.36 0.98 0.04
- link table_center: geometry collision box size=0.55 0.95 0.72; visual box size=0.55 0.95 0.72
Joints:
- joint shelf_back_piece_joint: origin xyz=0.36 0.515 0.75 rpy=0 0 0 -> xyz=0.36 0.49 0.75 rpy=0 0 0
- joint shelf_base_center_joint: origin xyz=0.18 0.515 0.0 rpy=0 0 0 -> xyz=0.18 0.49 0.0 rpy=0 0 0
- joint shelf_center_joint: origin xyz=0.18 0.515 0.75 rpy=0 0 0 -> xyz=0.18 0.49 0.75 rpy=0 0 0
- joint shelf_floor_1_piece_joint: origin xyz=0.0 0.0 0.347 rpy=0 0 0 -> xyz=0.0 0.0 0.43 rpy=0 0 0
- joint shelf_left_side_piece_joint: origin xyz=0.18 1.03 0.75 rpy=0 0 0 -> xyz=0.18 0.98 0.75 rpy=0 0 0
- joint shelf_origin_joint: origin xyz=0.0 0.0 0.0 rpy=0 0 0.0 -> xyz=0.0 0.05 0.0 rpy=0 0 -0.05
- joint table_center_joint: origin xyz=0.425 0.425 0.38 rpy=0 0 0 -> xyz=0.275 0.475 0.36 rpy=0 0 0
- joint table_front_edge_center_joint: origin xyz=0 0.425 0.76 rpy=0 0 0 -> xyz=0 0.475 0.72 rpy=0 0 0
- joint table_origin_joint: origin xyz=-0.12 1.45 0.0 rpy=0 0 1.570796 -> xyz=-1.28 -1.43 0.0 rpy=0 0 -1.655
- joint table_surface_center_joint: origin xyz=0.425 0.425 0.76 rpy=0 0 0 -> xyz=0.275 0.475 0.72 rpy=0 0 0

Commit message: last demo setup at iai

File: iai_hsr_robocup/urdf/HSR_robocup.urdf (robot description, URDF)
Before this commit: robot kitchen_description, 16 links, 15 joints
Links:
- link table_center: geometry collision box size=0.55 0.75 0.46; visual box size=0.55 0.75 0.46
Joints:
- joint table_center_joint: origin xyz=0.275 0.475 0.36 rpy=0 0 0 -> xyz=0.275 0.375 0.23 rpy=0 0 0
- joint table_front_edge_center_joint: origin xyz=0 0.475 0.72 rpy=0 0 0 -> xyz=0 0.375 0.46 rpy=0 0 0
- joint table_origin_joint: origin xyz=-1.28 -1.43 0.0 rpy=0 0 -1.655 -> xyz=-0.35 1.5 0.0 rpy=0 0 1.5
- joint table_surface_center_joint: origin xyz=0.275 0.475 0.72 rpy=0 0 0 -> xyz=0.275 0.375 0.46 rpy=0 0 0

Commit message: Set living room as default. Add OWL exporter scritp

File: iai_hsr_robocup/urdf/HSR_robocup.urdf (robot description, URDF)
Before this commit: robot kitchen_description, 16 links, 15 joints
Links:
- removed link shelf_floor_4_piece
- link shelf_back_piece: geometry collision box size=0.01 0.92 2.1; visual box size=0.01 0.92 2.1
- link shelf_floor_0_piece: geometry collision box size=0.4 0.92 0.04; visual box size=0.4 0.92 0.04
- link shelf_floor_1_piece: geometry collision box size=0.4 0.92 0.04; visual box size=0.4 0.92 0.04
- link shelf_floor_2_piece: geometry collision box size=0.4 0.92 0.04; visual box size=0.4 0.92 0.04
- link shelf_floor_3_piece: geometry collision box size=0.4 0.92 0.04; visual box size=0.4 0.92 0.04
- link shelf_left_side_piece: geometry collision box size=0.4 0.01 2.1; visual box size=0.4 0.01 2.1
- link shelf_right_side_piece: geometry collision box size=0.4 0.01 2.1; visual box size=0.4 0.01 2.1
Joints:
- removed joint shelf_floor_4_piece_joint
- joint shelf_back_piece_joint: origin xyz=0.36 0.49 0.75 rpy=0 0 0 -> xyz=0.4 0.46 1.05 rpy=0 0 0
- joint shelf_base_center_joint: origin xyz=0.18 0.49 0.0 rpy=0 0 0 -> xyz=0.2 0.46 0.0 rpy=0 0 0
- joint shelf_center_joint: origin xyz=0.18 0.49 0.75 rpy=0 0 0 -> xyz=0.2 0.46 1.05 rpy=0 0 0
- joint shelf_floor_0_piece_joint: origin xyz=0.0 0.0 0.06 rpy=0 0 0 -> xyz=0.0 0.0 0.1 rpy=0 0 0
- joint shelf_floor_1_piece_joint: origin xyz=0.0 0.0 0.43 rpy=0 0 0 -> xyz=0.0 0.0 0.41 rpy=0 0 0
- joint shelf_floor_2_piece_joint: origin xyz=0.0 0.0 0.8 rpy=0 0 0 -> xyz=0.0 0.0 0.77 rpy=0 0 0
- joint shelf_floor_3_piece_joint: origin xyz=0.0 0.0 1.162 rpy=0 0 0 -> xyz=0.0 0.0 1.05 rpy=0 0 0
- joint shelf_left_side_piece_joint: origin xyz=0.18 0.98 0.75 rpy=0 0 0 -> xyz=0.2 0.92 1.05 rpy=0 0 0
- joint shelf_origin_joint: origin xyz=0.0 0.05 0.0 rpy=0 0 -0.05 -> xyz=0.0 -0.1 0.0 rpy=0 0 -0.05
- joint shelf_right_side_piece_joint: origin xyz=0.18 0.0 0.75 rpy=0 0 0 -> xyz=0.2 0.0 1.05 rpy=0 0 0
- joint table_origin_joint: origin xyz=-0.35 1.5 0.0 rpy=0 0 1.5 -> xyz=-1.62 0.57 0.0 rpy=0 0 1.5

Commit message: Back home in the IAI lab again

File: iai_hsr_robocup/urdf/HSR_robocup.urdf (robot description, URDF)
Before this commit: robot kitchen_description, 15 links, 14 joints
Links:
- added link shelf_floor_4_piece; collision box size=0.36 0.98 0.04; visual box size=0.36 0.98 0.04
- link shelf_back_piece: geometry collision box size=0.01 0.98 1.5; visual box size=0.01 0.98 1.5
- link shelf_floor_0_piece: geometry collision box size=0.36 0.98 0.04; visual box size=0.36 0.98 0.04
- link shelf_floor_1_piece: geometry collision box size=0.36 0.98 0.04; visual box size=0.36 0.98 0.04
- link shelf_floor_2_piece: geometry collision box size=0.36 0.98 0.04; visual box size=0.36 0.98 0.04
- link shelf_floor_3_piece: geometry collision box size=0.36 0.98 0.04; visual box size=0.36 0.98 0.04
- link shelf_left_side_piece: geometry collision box size=0.36 0.01 1.5; visual box size=0.36 0.01 1.5
- link shelf_right_side_piece: geometry collision box size=0.36 0.01 1.5; visual box size=0.36 0.01 1.5
- link table_center: geometry collision box size=0.55 0.95 0.72; visual box size=0.55 0.95 0.72
Joints:
- added joint shelf_floor_4_piece_joint: type fixed, parent shelf_base_center, child shelf_floor_4_piece, origin xyz=0.0 0.0 1.478 rpy=0 0 0
- joint shelf_back_piece_joint: origin xyz=0.4 0.46 1.05 rpy=0 0 0 -> xyz=0.36 0.49 0.75 rpy=0 0 0
- joint shelf_base_center_joint: origin xyz=0.2 0.46 0.0 rpy=0 0 0 -> xyz=0.18 0.49 0.0 rpy=0 0 0
- joint shelf_center_joint: origin xyz=0.2 0.46 1.05 rpy=0 0 0 -> xyz=0.18 0.49 0.75 rpy=0 0 0
- joint shelf_floor_0_piece_joint: origin xyz=0.0 0.0 0.1 rpy=0 0 0 -> xyz=0.0 0.0 0.06 rpy=0 0 0
- joint shelf_floor_1_piece_joint: origin xyz=0.0 0.0 0.41 rpy=0 0 0 -> xyz=0.0 0.0 0.43 rpy=0 0 0
- joint shelf_floor_2_piece_joint: origin xyz=0.0 0.0 0.77 rpy=0 0 0 -> xyz=0.0 0.0 0.8 rpy=0 0 0
- joint shelf_floor_3_piece_joint: origin xyz=0.0 0.0 1.05 rpy=0 0 0 -> xyz=0.0 0.0 1.162 rpy=0 0 0
- joint shelf_left_side_piece_joint: origin xyz=0.2 0.92 1.05 rpy=0 0 0 -> xyz=0.18 0.98 0.75 rpy=0 0 0
- joint shelf_origin_joint: origin xyz=0.0 -0.1 0.0 rpy=0 0 -0.05 -> xyz=0.0 0.05 0.0 rpy=0 0 -0.05
- joint shelf_right_side_piece_joint: origin xyz=0.2 0.0 1.05 rpy=0 0 0 -> xyz=0.18 0.0 0.75 rpy=0 0 0
- joint table_center_joint: origin xyz=0.275 0.375 0.23 rpy=0 0 0 -> xyz=0.275 0.475 0.36 rpy=0 0 0
- joint table_front_edge_center_joint: origin xyz=0 0.375 0.46 rpy=0 0 0 -> xyz=0 0.475 0.72 rpy=0 0 0
- joint table_origin_joint: origin xyz=-1.62 0.57 0.0 rpy=0 0 1.5 -> xyz=-1.28 -1.43 0.0 rpy=0 0 -1.655
- joint table_surface_center_joint: origin xyz=0.275 0.375 0.46 rpy=0 0 0 -> xyz=0.275 0.475 0.72 rpy=0 0 0
